File: PCBusinessCard/NFC_BusinessCard.kicad_pcb (KiCad board)
At the start: 2 copper layers, 85.6 x 68.1 mm, 20 parts

Commit message: testing kicad 7 branch
Other:
- board text added: "1-833-GHLOPEZ"

Commit message: contact info changed
Other:
- board text added: "PH: 1-833-GHLOPEZ"
- board text added: "SMS: 1-833-445-6739"
- board text added: "glennlopez.com"
- board text added: "me@glennlopez.com"
- board text removed: "1-833-GHLOPEZ"
